Commit message: PhaseTwo

File: urdf/base.xacro (robot description, xacro)
@@ -53,8 +53,24 @@
        the STEP says 30.000 mm and the STEP wins. See README. -->
   <xacro:property name="wheel_z" value="${wheel_radius - base_link_height}"/>
-  <!-- Emit <inertial> blocks? Off by default: the chassis mass properties are
-       not yet supplied and this package will not invent them. See
-       inertial_macros.xacro and the TODO block further down. -->
-  <xacro:property name="use_inertial" value="false"/>
+  <!-- Emit <inertial> blocks?
+       Phase 1 default was false: no mass properties had been supplied and the
+       brief forbids placeholder tensors, so RViz got a description with no
+       invented numbers in it.
+       Phase 2 default is TRUE, because Gazebo cannot simulate a link without
+       an inertial. The tensors are NOT placeholders and NOT identity - they
+       are integrated from the real collision geometry by
+       tools/estimate_inertia.py. Read that file's docstring before trusting
+       them: the SHAPE of every tensor is exact geometry, the SCALE depends on
+       a mass, and only two of the three masses have a source.
+       Set false to get the Phase 1 behaviour back. -->
+  <xacro:property name="use_inertial" value="true"/>
+  <!-- Masses. PROVENANCE MATTERS HERE - see README "Inertials".
+       chassis : GIVEN in the brief, section 3.1.
+       wheel   : *** THE ONE UNSOURCED NUMBER IN THIS PACKAGE. ***
+                 Not measured, not from a datasheet. It exists so the sim runs.
+                 Weigh one wheel and replace it. Wheel inertia sets drive
+                 acceleration, so a wrong value reads as a tuning problem. -->
+  <xacro:property name="chassis_mass" value="1.0"/>
+  <xacro:property name="wheel_mass"   value="0.100"/>   <!-- TODO(weigh me) -->
   <xacro:property name="deg" value="${pi/180.0}"/>
   <xacro:property name="mesh_visual"    value="package://mmr_pkg/meshes/visual"/>
@@ -123,14 +139,22 @@
       </geometry>
     </collision>
-    <!-- TODO(inertial): chassis mass excluding arm, Pi and battery is 1.0 kg
-         per the brief, but CoM and the inertia tensor are not yet supplied.
-         Paste the Fusion 360 physical-properties numbers into
-         inertial_macros.xacro's inertial_from_fusion and set
-         use_inertial to true. No placeholder tensor is emitted here. -->
+    <!-- Inertia integrated from the collision set above (two plate cylinders,
+         three motor pods, camera pod, Pi stack) at one uniform density scaled
+         to the brief's 1.0 kg, combined by the parallel-axis theorem.
+         Regenerate with `python tools/estimate_inertia.py`.
+         The visual mesh is deliberately NOT used: it is a decimated CAD export
+         and is not watertight, so a volume integral over it is meaningless
+         (trimesh returns a number regardless, which is the trap).
+         Resulting CoM (-0.3, -0.0, +21.8) mm - essentially centred and low,
+         as expected for a heavy base plate. Radius of gyration 88.9 mm
+         against a 120 mm plate radius.
+         Still an approximation: one density across plates, Pi and motors. If
+         you paste real Fusion numbers, use inertial_from_fusion instead - it
+         handles the kg*mm^2 and product-of-inertia sign conversions. -->
     <xacro:if value="${use_inertial}">
-      <!-- <xacro:inertial_from_fusion mass="1.0"
-             ixx="TODO" iyy="TODO" izz="TODO"
-             ixy="TODO" ixz="TODO" iyz="TODO"
-             com_x_mm="TODO" com_y_mm="TODO" com_z_mm="TODO"/> -->
+      <xacro:inertial_exact mass="${chassis_mass}"
+          ox="-0.000277" oy="-0.000032" oz="0.021827"
+          ixx="0.004760788" iyy="0.005840846" izz="0.007861537"
+          ixy="0.000000057" ixz="0.000351742" iyz="0.000001738"/>
     </xacro:if>
   </link>
@@ -170,8 +194,10 @@
         </geometry>
       </collision>
-      <!-- TODO(inertial): per-wheel mass not supplied. See base_link. -->
+      <!-- Solid cylinder about local +X, exact for the modelled collision
+           shape. The MASS is the unsourced number - see the wheel_mass
+           property at the top of this file. -->
       <xacro:if value="${use_inertial}">
-        <!-- <xacro:inertial_cylinder_x mass="TODO"
-               radius="${wheel_radius}" length="${wheel_width}"/> -->
+        <xacro:inertial_cylinder_x mass="${wheel_mass}"
+               radius="${wheel_radius}" length="${wheel_width}"/>
       </xacro:if>
     </link>

File: urdf/mmr_bot.urdf.xacro (robot description, xacro)
@@ -20,5 +20,23 @@
 <!-- 14 links, 13 joints, of which 9 are movable (3 wheels + 6 arm).         -->
 <!-- ====================================================================== -->
-<robot name="mmr_bot" xmlns:xacro="http://www.ros.org/wiki/xacro">
+<!-- xmlns:gz is required by the omniwheel friction block in gazebo.xacro,
+     which uses gz:expressed_in on <fdir1> to pin the roller axis to the
+     chassis frame instead of the (spinning) wheel frame. Declared here at the
+     root because that is the only place a namespace declaration survives
+     xacro expansion into the final URDF. -->
+<robot name="mmr_bot"
+       xmlns:xacro="http://www.ros.org/wiki/xacro"
+       xmlns:gz="http://gazebosim.org/schema">
+  <!-- ==================================================================== -->
+  <!-- Phase 2 toggles.                                                     -->
+  <!--                                                                      -->
+  <!--   ros2 run xacro xacro mmr_bot.urdf.xacro                (sim, full)  -->
+  <!--   ros2 run xacro xacro mmr_bot.urdf.xacro gazebo:=false  (Phase 1)    -->
+  <!--                                                                      -->
+  <!-- gazebo:=false reproduces the Phase 1 description byte-for-byte apart  -->
+  <!-- from the xmlns:gz attribute, so display.launch.py and anything that   -->
+  <!-- only wants geometry are unaffected by Phase 2.                        -->
+  <!-- ==================================================================== -->
+  <xacro:arg name="gazebo" default="true"/>
   <xacro:include filename="$(find mmr_pkg)/urdf/inertial_macros.xacro"/>
   <xacro:include filename="$(find mmr_pkg)/urdf/base.xacro"/>
@@ -44,3 +62,19 @@
     <origin xyz="${arm_mount_x} ${arm_mount_y} ${arm_mount_z}" rpy="0 0 0"/>
   </xacro:so101_arm>
+  <!-- ================================================================== -->
+  <!-- Phase 2: simulation.                                                -->
+  <!--                                                                     -->
+  <!-- Both files are included INSIDE the gazebo guard. ros2_control.xacro  -->
+  <!-- is guarded too, not just gazebo.xacro, because its only hardware     -->
+  <!-- plugin today is the Gazebo one - there is no ESP32                   -->
+  <!-- hardware_interface yet (see the TODO in that file). When one is      -->
+  <!-- written this include moves out of the guard and the `sim` parameter  -->
+  <!-- of mmr_ros2_control starts earning its keep.                         -->
+  <!-- ================================================================== -->
+  <xacro:if value="$(arg gazebo)">
+    <xacro:include filename="$(find mmr_pkg)/urdf/ros2_control.xacro"/>
+    <xacro:include filename="$(find mmr_pkg)/urdf/gazebo.xacro"/>
+    <xacro:mmr_ros2_control sim="true"/>
+    <xacro:mmr_gazebo/>
+  </xacro:if>
 </robot>

File: urdf/sensors.xacro (robot description, xacro)
@@ -9,13 +9,22 @@
        CAD (0.200, -133.78) mm, giving 133.781 mm forward of base_link and
        0.004 mm off centre (i.e. on the forward axis to within 4 microns).
-       TODO(confirm z): 0.105180 m is the MID-HEIGHT of the turret shell
-       (CAD z 137.000..163.241 mm). The true optical/scan plane of an RPLIDAR
-       C1 is not derivable from this STEP - the CAD body is a solid shell with
-       no modelled optics. If you want the scan plane exactly, measure from
-       the datasheet and override laser_z below. Everything else in this file
-       is measured, this one number is a documented approximation. -->
+       z RESOLVED in Phase 2 from the datasheet, no longer a guess. The
+       Slamtec C1 mechanical drawing (rev 1.2, Fig 4-1) dimensions the
+       "Laser Receiving and Emitting Height" at 29.800 mm above the bottom
+       mounting face. The collision hull's lowest face is a genuinely planar
+       48-vertex surface at -28.179 mm in this frame, spanning exactly
+       +/-27.800 mm in x and y, which is the datasheet's 55.6 mm mounting
+       base. So:
+           scan plane = -28.179 + 29.800 = +1.621 mm from the mesh origin
+           laser_z    =  0.105180 + 0.001621 = 0.106801 m
+       Cross-check: that puts the mounting face at base_link z = 0.077001 m,
+       which is the top plate's upper surface (top_plate_z 0.072 + 0.005
+       thickness) to within 1 micron. The lidar bolts to the top plate, as
+       drawn. The Phase 1 turret-mid-height guess was low by 1.621 mm.
+       Body bbox also confirms the mesh: 55.6 x 41.3 mm matches the
+       datasheet exactly (the 64.8 mm x span is body + UART connector). -->
   <xacro:property name="laser_x" value="0.133781"/>
   <xacro:property name="laser_y" value="0.000004"/>
-  <xacro:property name="laser_z" value="0.105180"/>
+  <xacro:property name="laser_z" value="0.106801"/>
   <!-- rpy is identity: the lidar body is axis-aligned with base_link in CAD,
        and the C1 scans in its own XY plane with zero angle at its +X. -->
@@ -42,6 +51,14 @@
       </geometry>
     </collision>
-    <!-- TODO(inertial): RPLIDAR C1 mass not supplied. Datasheet value or a
-         Fusion physical-properties readout would fill this. Not invented. -->
+    <!-- Mass 110 g is the datasheet's typical figure (rev 1.2, Fig 2-9), so
+         this one is sourced. The tensor is a uniform-density integral over the
+         convex hull; the real unit is denser at the motor end, but the hull
+         has the right outline and the part is small enough that the error is
+         not going to change how the robot behaves.
+         Regenerate with tools/estimate_inertia.py. -->
+    <xacro:inertial_exact mass="0.110"
+        ox="-0.001128" oy="-0.000003" oz="-0.009419"
+        ixx="0.000037988" iyy="0.000041294" izz="0.000050888"
+        ixy="0.0" ixz="-0.000000835" iyz="0.0"/>
   </link>
   <!-- NOTE: the brief says "no cameras yet", but the STEP does model one:
